File: v0.2/voltage_sensor_v0.2.sch (EAGLE design)
At the start: 56 parts, among them IC1 AP2112K-3.3TRG1, J2 236-404_000-009_999-950, J3 MC000048, J9 RJ11, T1 ZMPT101B, T2 ZMPT101B, T3 ZMPT101B

Commit message: fix resistor footprint and value
Parts:
- R1, R12, R15, R16, R17, R18, R19, R2, R25, R26, R27, R28, R29, R3, R30, R4, R5, R6: value (none) -> 10k; device rcl:R-EU_R1206 -> rcl:R-EU_R0603
- R21, R8, R9: value (none) -> 75R; device rcl:R-EU_R1206 -> rcl:R-EU_R0603
