File: v0.4/voltage_sensor_v0.4.brd (EAGLE design)
At the start: 77 x 100 mm, 59 parts, among them IC1 AP2112K-3.3TRG1, J1 1017505, J2 20020316-H021B01LF, J9 RJ11-6, M1 MOV-14D431KTR, M2 MOV-14D431KTR, M3 MOV-14D431KTR, T1 ZMPT101B, T2 ZMPT101B, T3 ZMPT101B

Commit message: fix PSU 10W footprint
Connections:
- net 5V: now also PS1.4; no longer PS1.6
- net GND: now also PS1.6; no longer PS1.4
Routing:
- net 5V: track 144.4 -> 133.9 mm, vias 2 -> 1
- net GND: track 215.2 -> 219.1 mm
Changed lines of the file:
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@@
 <vertex x="7" y="106"/>
 </polygon>
-<contactref element="PS1" pad="4"/>
 <contactref element="PS2" pad="4"/>
 <contactref element="IC1" pad="4"/>
@@
 <contactref element="C5" pad="-"/>
 <contactref element="D1" pad="2"/>
-<wire x1="58.15" y1="5.8" x2="58.15" y2="11.835" width="1.016" layer="1"/>
-<wire x1="58.15" y1="11.835" x2="59.295" y2="12.98" width="1.016" layer="1"/>
 <wire x1="46.75" y1="3.3" x2="46.4" y2="3.65" width="1.016" layer="1"/>
 <wire x1="58.42" y1="5.53" x2="58.42" y2="4.064" width="1.016" layer="1"/>
@@
 <wire x1="19.088" y1="7.112" x2="19.25" y2="6.95" width="0.508" layer="1"/>
 <wire x1="2.54" y1="27.94" x2="2.54" y2="36.084" width="0.508" layer="16"/>
-<wire x1="59.295" y1="14.815" x2="59.295" y2="12.98" width="1.27" layer="16"/>
-<wire x1="73.32" y1="28.84" x2="59.295" y2="14.815" width="1.27" layer="16"/>
 <via x="15.748" y="42.164" extent="1-16" drill="0.5"/>
 <via x="14.224" y="61.468" extent="1-16" drill="0.5"/>
@@
 <wire x1="15" y1="2.808" x2="15" y2="3.65" width="0.508" layer="1"/>
 <via x="26.216" y="6.024" extent="1-16" drill="0.5"/>
+<contactref element="PS1" pad="6"/>
+<wire x1="58.15" y1="5.8" x2="61.85" y2="9.5" width="1.016" layer="1"/>
+<wire x1="68.52" y1="9.5" x2="72" y2="12.98" width="1.016" layer="1"/>
+<wire x1="61.85" y1="9.5" x2="68.52" y2="9.5" width="1.016" layer="1"/>
+<wire x1="72" y1="12.98" x2="73.32" y2="14.3" width="1.016" layer="1"/>
+<wire x1="73.32" y1="14.3" x2="73.32" y2="28.84" width="1.016" layer="1"/>
 </signal>
 <signal name="N$25">
@@
 <signal name="5V">
 <contactref element="J9" pad="2"/>
-<contactref element="PS1" pad="6"/>
 <contactref element="PS2" pad="5"/>
 <contactref element="C3" pad="1"/>
@@
 <contactref element="C6" pad="1"/>
 <contactref element="D1" pad="1"/>
-<wire x1="72" y1="12.98" x2="70.612" y2="14.368" width="1.27" layer="1"/>
 <wire x1="70.612" y1="36.292" x2="73.32" y2="39" width="1.27" layer="1"/>
-<wire x1="70.612" y1="14.368" x2="70.612" y2="36.292" width="1.27" layer="1"/>
 <wire x1="56.45" y1="5.8" x2="55.668" y2="5.8" width="1.016" layer="1"/>
 <wire x1="21.75" y1="5.05" x2="23.906" y2="5.05" width="0.508" layer="1"/>
 <wire x1="52.8" y1="6.95" x2="52.832" y2="6.532" width="1.27" layer="1"/>
-<wire x1="52.832" y1="6.532" x2="52.832" y2="9.652" width="1.27" layer="1"/>
-<via x="52.832" y="9.652" extent="1-16" drill="0.5"/>
-<wire x1="52.832" y1="9.652" x2="68.672" y2="9.652" width="1.27" layer="16"/>
-<wire x1="68.672" y1="9.652" x2="72" y2="12.98" width="1.27" layer="16"/>
 <wire x1="46.4" y1="7.95" x2="51.35" y2="7.95" width="1.27" layer="1"/>
 <wire x1="51.35" y1="7.95" x2="52.8" y2="6.95" width="1.27" layer="1"/>
@@
 <wire x1="31" y1="7.5" x2="33" y2="5.5" width="0.508" layer="1"/>
 <wire x1="33" y1="5.5" x2="33" y2="3.5" width="0.508" layer="1"/>
+<contactref element="PS1" pad="4"/>
+<wire x1="59.295" y1="12.98" x2="59.295" y2="22.295" width="1.27" layer="1"/>
+<wire x1="70.612" y1="33.612" x2="70.612" y2="36.292" width="1.27" layer="1"/>
+<wire x1="59.295" y1="22.295" x2="70.612" y2="33.612" width="1.27" layer="1"/>
+<wire x1="59.295" y1="12.98" x2="53.265" y2="6.95" width="1.27" layer="1"/>
+<wire x1="53.265" y1="6.95" x2="52.8" y2="6.95" width="1.27" layer="1"/>
 </signal>
 <signal name="N$17">

Commit message: fiducials
Parts:
- removed U$1, U$2, U$3: (no value), special:DRIL-2
- added FD1, FD2, FD3: FIDUCIAL1X2, SparkFun-Aesthetics:FIDUCIAL-1X2
- added LOGO1: ROHS_LOGO, SparkFun-Aesthetics:ROHS_LOGO_0.18_IN
- added LOGO2: OSHW-LOGOS-COPPER, SparkFun-Aesthetics:OSHW-LOGO-S_COPPER
Routing:
- net GND: track 219.1 -> 218.5 mm
Changed lines of the file:
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@@
 <attribute name="VALUE" x="70.025" y="58.04" size="1.27" layer="27" rot="R270"/>
 </element>
-<element name="U$1" library="special" library_urn="urn:adsk.eagle:library:367" package="DRIL-2" value="" x="65" y="3.5" smashed="yes"/>
-<element name="U$2" library="special" library_urn="urn:adsk.eagle:library:367" package="DRIL-2" value="" x="4" y="13" smashed="yes"/>
-<element name="U$3" library="special" library_urn="urn:adsk.eagle:library:367" package="DRIL-2" value="" x="72.3" y="92.9" smashed="yes"/>
 <element name="J1" library="1017505" package="1017505" value="1017505" x="59.1" y="78.5" smashed="yes" rot="R180">
 <attribute name="ARROW_PART_NUMBER" value="1017505" x="59.1" y="78.5" size="1.778" layer="27" rot="R180" display="off"/>
@@
 <attribute name="VALUE" x="41.92" y="19.85" size="1.27" layer="27" align="center"/>
 </element>
+<element name="FD1" library="SparkFun-Aesthetics" package="FIDUCIAL-1X2" value="FIDUCIAL1X2" x="3.5" y="11.5" smashed="yes"/>
+<element name="FD2" library="SparkFun-Aesthetics" package="FIDUCIAL-1X2" value="FIDUCIAL1X2" x="65.5" y="3.5" smashed="yes"/>
+<element name="FD3" library="SparkFun-Aesthetics" package="FIDUCIAL-1X2" value="FIDUCIAL1X2" x="72.5" y="93.5" smashed="yes"/>
+<element name="LOGO1" library="SparkFun-Aesthetics" package="ROHS_LOGO_0.18_IN" value="ROHS_LOGO" x="68.5" y="81.5" smashed="yes"/>
+<element name="LOGO2" library="SparkFun-Aesthetics" package="OSHW-LOGO-S_COPPER" value="OSHW-LOGOS-COPPER" x="70.5" y="78.5" smashed="yes"/>
 </elements>
 <signals>
@@
 <wire x1="17.272" y1="7.112" x2="19.088" y2="7.112" width="0.508" layer="1"/>
 <wire x1="19.088" y1="7.112" x2="19.25" y2="6.95" width="0.508" layer="1"/>
-<wire x1="2.54" y1="27.94" x2="2.54" y2="36.084" width="0.508" layer="16"/>
 <via x="15.748" y="42.164" extent="1-16" drill="0.5"/>
 <via x="14.224" y="61.468" extent="1-16" drill="0.5"/>
@@
 <wire x1="11.176" y1="11.676" x2="14" y2="14.5" width="0.508" layer="16"/>
 <wire x1="14" y1="14.5" x2="14" y2="17.5" width="0.508" layer="16"/>
-<wire x1="3.56" y1="27.94" x2="2.54" y2="27.94" width="0.508" layer="16"/>
-<wire x1="14" y1="17.5" x2="3.56" y2="27.94" width="0.508" layer="16"/>
 <wire x1="12" y1="3.65" x2="10.35" y2="3.65" width="0.508" layer="1"/>
 <wire x1="10.35" y1="3.65" x2="10" y2="4" width="0.508" layer="1"/>
@@
 <wire x1="72" y1="12.98" x2="73.32" y2="14.3" width="1.016" layer="1"/>
 <wire x1="73.32" y1="14.3" x2="73.32" y2="28.84" width="1.016" layer="1"/>
+<wire x1="2.54" y1="28.96" x2="2.54" y2="36.084" width="0.508" layer="16"/>
+<wire x1="14" y1="17.5" x2="2.54" y2="28.96" width="0.508" layer="16"/>
+<wire x1="14.224" y1="79.756" x2="16.224" y2="91.608" width="0" layer="19" extent="1-1"/>
+<wire x1="2.706" y1="80.28" x2="14.224" y2="79.756" width="0" layer="19" extent="1-1"/>
+<wire x1="49.784" y1="1.524" x2="52.8" y2="2.85" width="0" layer="19" extent="1-1"/>
+<wire x1="55.88" y1="1.524" x2="52.8" y2="2.85" width="0" layer="19" extent="1-1"/>
+<wire x1="26.216" y1="6.024" x2="24.22" y2="9.31" width="0" layer="19" extent="1-1"/>
+<wire x1="3.048" y1="90.424" x2="2.706" y2="80.28" width="0" layer="19" extent="1-1"/>
+<wire x1="14.224" y1="61.468" x2="2.706" y2="61.484" width="0" layer="19" extent="1-1"/>
+<wire x1="15.748" y1="42.164" x2="2.706" y2="42.18" width="0" layer="19" extent="1-1"/>
 </signal>
 <signal name="N$25">

Commit message: add filter components
Parts:
- added C4: B32923C3105M000, B32923C3105M000:B32923C_(26.5_X_12)
- added U$1: 47mH, Schaffner-CM-Choke:RN114-0.3-02-47M
- added U$2: RN214-0.3-02-47M, Schaffner-CM-Choke:RN214-0.3-02-47M
Changed lines of the file:
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@@
 <element name="LOGO1" library="SparkFun-Aesthetics" package="ROHS_LOGO_0.18_IN" value="ROHS_LOGO" x="68.5" y="81.5" smashed="yes"/>
 <element name="LOGO2" library="SparkFun-Aesthetics" package="OSHW-LOGO-S_COPPER" value="OSHW-LOGOS-COPPER" x="70.5" y="78.5" smashed="yes"/>
+<element name="U$2" library="Schaffner-CM-Choke" package="RN214-0.3-02-47M" value="RN214-0.3-02-47M" x="58" y="87" smashed="yes"/>
+<element name="U$1" library="Schaffner-CM-Choke" package="RN114-0.3-02-47M" value="47mH" x="43.5" y="93.5" smashed="yes"/>
+<element name="C4" library="B32923C3105M000" package="B32923C_(26.5_X_12)" value="B32923C3105M000" x="2" y="-9.5" smashed="yes">
+<attribute name="ARROW_PART_NUMBER" value="B32923C3105M000" x="2" y="-9.5" size="1.778" layer="27" display="off"/>
+<attribute name="ARROW_PRICE-STOCK" value="https://www.arrow.com/en/products/b32923c3105m000/epcos-tdk" x="2" y="-9.5" size="1.778" layer="27" display="off"/>
+<attribute name="DESCRIPTION" value="EPCOS - B32923C3105M000 - Safety Capacitor, 1 ?F, X2, B32923C Series, 305 V, Metallized PP" x="2" y="-9.5" size="1.778" layer="27" display="off"/>
+<attribute name="HEIGHT" value="mm" x="2" y="-9.5" size="1.778" layer="27" display="off"/>
+<attribute name="MANUFACTURER_NAME" value="TDK" x="2" y="-9.5" size="1.778" layer="27" display="off"/>
+<attribute name="MANUFACTURER_PART_NUMBER" value="B32923C3105M000" x="2" y="-9.5" size="1.778" layer="27" display="off"/>
+<attribute name="MOUSER_PART_NUMBER" value="" x="2" y="-9.5" size="1.778" layer="27" display="off"/>
+<attribute name="MOUSER_PRICE-STOCK" value="" x="2" y="-9.5" size="1.778" layer="27" display="off"/>
+<attribute name="NAME" x="2" y="-9.5" size="1.27" layer="25" align="center"/>
+<attribute name="VALUE" x="2" y="-9.5" size="1.27" layer="27" align="center"/>
+</element>
 </elements>
 <signals>
