File: v0.5/voltage_sensor_v0.5.brd (EAGLE design)
At the start: 73 x 118 mm, 64 parts, among them IC1 AP2112K-3.3TRG1, J1 1017505, J2 20020316-H021B01LF, J9 RJ11-6, M1 MOV-14D431KTR, M2 MOV-14D431KTR, M3 MOV-14D431KTR, T1 ZMPT101B, T2 ZMPT101B, T3 ZMPT101B

Commit message: new design
Parts:
- removed J1: 1017505, 1017505:1017505
- removed R34: 12R 3W, rcl:R2512
- added U$3, U$5, U$6, U$7, U$8: 1905010, Phoenix-Contact-1905010:1905010
- moved C4 51.8 mm to (41.4, 57.7), turned to 90 degrees
- moved U$1 28.6 mm to (61.5, 82.0), turned to 90 degrees
- moved JP1 27.7 mm to (20.5, 10.0)
- moved U$2 27.5 mm to (72.5, 74.0), turned to 90 degrees
- moved C9 26.2 mm to (36.0, 10.0)
- moved C7 25.7 mm to (38.6, 10.0)
- moved C6 24.7 mm to (45.7, 9.96)
- moved IC1 24.0 mm to (42.0, 10.0)
- moved R29 21.8 mm to (21.6, 80.4)
- moved R28 21.0 mm to (17.0, 80.9)
- moved R30 20.1 mm to (25.7, 81.3)
- moved F3 19.9 mm to (26.3, 93.1)
- moved T3 19.5 mm to (22.9, 62.2)
- moved F2 19.0 mm to (32.4, 93.1)
- moved FD1 19.0 mm to (12.5, 5.00)
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Connections:
- net GND: now also U$7.P$1, U$7.P$2
- net L1: now also PS1.1, PS2.2, U$1.P$3, U$2.P$3; no longer F1.OUT, R34.1
- net N$16: now also U$8.P$1, U$8.P$2; no longer J1.7, J1.8
- net N$17: now also C4.2, F1.OUT, U$1.P$4, U$2.P$4; no longer PS1.1, PS2.2, R34.2
- net N$7: now also U$5.P$1, U$5.P$2; no longer J1.3, J1.4
- net N$8: now also U$3.P$1, U$3.P$2; no longer J1.5, J1.6
- net NEUTRAL: now also C4.1, U$1.P$1, U$1.P$2, U$2.P$1, U$2.P$2, U$6.P$1, U$6.P$2; no longer J1.1, J1.2
Other:
- board size 73 x 118 mm -> 73 x 113 mm
- board text added: "emonVS"
- board text removed: "emonVoltageSense"

Commit message: finish layout
Parts:
- added C10: DE2F3KY103MA3BM02F, DE2F3KY103MA3BM02F:DE2F3KY103MA3BM02F
- moved R28 17.1 mm to (30.0, 69.6)
- moved R27 15.7 mm to (30.0, 67.1)
- moved R26 14.2 mm to (30.0, 64.5)
- moved R19 12.9 mm to (30.0, 57.9), turned to 0 degrees
- moved R25 12.7 mm to (30.0, 62.0)
- moved R29 11.7 mm to (30.0, 72.1), turned to 180 degrees
- moved R18 11.2 mm to (30.0, 55.4), turned to 180 degrees
- moved R17 9.74 mm to (30.0, 52.8)
- moved R16 8.19 mm to (30.0, 50.3)
- moved R30 7.91 mm to (30.0, 74.7), turned to 0 degrees
- moved R15 6.67 mm to (30.0, 47.8)
- moved R12 4.66 mm to (30.0, 45.2)
- moved R6 4.64 mm to (30.0, 41.1)
- moved R5 3.29 mm to (30.0, 38.6)
- moved R1 2.98 mm to (30.0, 28.4)
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- renumbered J2 to J6, J9 to J7, U$3 to J4, U$5 to J3, U$7 to J1, U$8 to J5
Connections:
- removed net N$18: C2.1, R20.1, R21.1, R23.1, R24.1, T3.3
- new net N$26: C8.1, R13.1, R14.1, R22.2, R9.2, T1.4
- net N$17: now also C10.2
- net N$25: now also C2.1, R20.2, R21.2, R23.1, R24.1, T3.4; no longer C8.1, R13.1, R14.1, R22.1, R9.1, T1.3
- net N$9: now also R7.2, R8.2, T2.4; no longer R7.1, R8.1, T2.3
- net NEUTRAL: now also C10.1
- net VS1: now also R22.1, R9.1, T1.3; no longer R22.2, R9.2, T1.4
- net VS2: now also R7.1, R8.1, T2.3; no longer R7.2, R8.2, T2.4
- net VS3: now also R20.1, R21.1, T3.3; no longer R20.2, R21.2, T3.4
Other:
- board text added: "J1"
- board text added: "J2"
- board text added: "J3"
- board text added: "J4"
- board text added: "J5"
- board text added: "J7"
- board text added: "U$1"

Commit message: v0.5 release
Parts:
- removed R20, R22, R7: (no value), rcl:0204/7
- removed U$2: RN214-0.3-02-47M, Schaffner-CM-Choke:RN214-0.3-02-47M
- added L1: 744252101, 744252101:744252101
- added R21B, R8B, R9B: (no value), rcl:0204/7
- added U$1B: RN214-0.3-02-47M, Schaffner-CM-Choke:RN214-0.3-02-47M
- moved LOGO1 64.6 mm to (2.02, 85.7)
- moved LOGO2 54.7 mm to (12.7, 89.8)
- moved JP1 27.0 mm to (4.39, 31.7), turned to 180 degrees
- moved C9 23.9 mm to (12.3, 12.9), turned to 90 degrees
- moved C7 23.6 mm to (15.2, 12.9), turned to 90 degrees
- moved IC1 23.1 mm to (19.1, 13.0)
- moved C6 22.6 mm to (23.4, 13.0)
- moved R14 7.56 mm to (3.56, 34.5), turned to 180 degrees
- moved C8 7.51 mm to (3.56, 42.7)
- moved R13 7.51 mm to (3.56, 38.6)
- moved M3 6.70 mm to (53.8, 54.4)
- moved D1 6.12 mm to (41.8, 17.0)
- moved C5 5.68 mm to (40.4, 11.6)
- moved R9 5.48 mm to (7.11, 39.1)
- moved C3 4.72 mm to (45.2, 10.7), turned to 270 degrees
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- renumbered PS2 to PS1B
Connections:
- removed net N$17: C10.2, C4.2, F1.OUT, U$1.P$4, U$2.P$4
- new net N$18: J7.2, L1.1
- new net N$27: J7.1, L1.3
- new net N$28: C10.1, C4.1, U$1.P$4, U$1B.P$4, U$6.P$1, U$6.P$2
- new net N$29: C10.2, C4.2, F1.OUT, U$1.P$2, U$1B.P$2
- net 5V: now also L1.6; no longer J7.2
- net GND: now also L1.4; no longer J7.1
- net L1: now also U$1.P$1, U$1B.P$1; no longer U$1.P$3, U$2.P$3
- net N$25: now also R21B.2; no longer R20.2
- net N$26: now also R9B.2; no longer R22.2
- net N$9: now also R8B.2; no longer R7.2
- net NEUTRAL: now also U$1.P$3, U$1B.P$3; no longer C10.1, C4.1, U$1.P$1, U$1.P$2, U$2.P$1, U$2.P$2, U$6.P$1, U$6.P$2
- net VS1: now also R9B.1; no longer R22.1
- net VS2: now also R8B.1; no longer R7.1
- net VS3: now also R21B.1; no longer R20.1
Routing:
- net GND: track 0.00 -> 284.5 mm, vias 0 -> 19
- net NEUTRAL: track 0.00 -> 110.6 mm
- net 5V: track 0.00 -> 103.1 mm, vias 0 -> 1
- net N$28: track 0.00 -> 86.7 mm
- net L1: track 0.00 -> 83.2 mm, vias 0 -> 1
- net L2: track 0.00 -> 82.2 mm, vias 0 -> 1
- net VS3: track 0.00 -> 74.7 mm
- net 3.3V: track 0.00 -> 73.5 mm
- net VS2: track 0.00 -> 65.5 mm
- net L3: track 0.00 -> 59.6 mm
- net VS1: track 0.00 -> 45.1 mm
- net BIAS: track 0.00 -> 43.7 mm, vias 0 -> 1
- net N$29: track 0.00 -> 39.1 mm
- net N$26: track 0.00 -> 21.5 mm
- net N$9: track 0.00 -> 20.1 mm
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Other:
- outline, holes or cut-outs redrawn
- board text added: "AC voltage sensing power supply"
- board text added: "Hardware"
- board text added: "Open"
- board text removed: "a"
- board text removed: "c"
