File: 1.3.2/emonVS.sch (EAGLE design)
At the start: 46 parts, among them CN1 TERMINAL_BLOCK_5P, CN2 RJ45 Jack, CN3 TERMINAL_BLOCK_2P, T1 ZMPT101B, T2 ZMPT101B, T3 ZMPT101B

Commit message: V1.3.2
Parts:
- removed C1: 1uF x 16V, My-RLC:C_0603
- removed L2: 100uH, OpenEnergyMonitor:CHOKES-WE-SL3
- added C4: 1uF x 310VAC, OpenEnergyMonitor:C_
- added U$1: 47mH, OpenEnergyMonitor:CHOKES-SCHAFFNER-RN214+RN212
- C3: value 1uF x 310VAC -> 1uF x 16V; device OpenEnergyMonitor:C_ -> My-RLC:C_0603; PN B32923C3105M000 -> GCM188R71C105KA64D
- L1: value 47mH -> 100uH; device OpenEnergyMonitor:CHOKES-SCHAFFNER-RN214+RN212 -> OpenEnergyMonitor:CHOKES-WE-SL3
- renumbered C2 to C5, CN1 to J9, CN2 to J7, CN3 to J8, RV1 to M1, RV2 to M2, RV3 to M3
Connections:
- net 5.0V: now also C3.1, L1.2; no longer C1.1, L2.2
- net 5VF: now also L1.1; no longer L2.1
- net GND: now also C3.2, L1.4; no longer C1.2, L2.4
- net GNDF: now also L1.3; no longer L2.3
- net L1_VOLTAGE: now also U$1.2; no longer L1.2
- net N$28: now also C4.2, U$1.3; no longer C3.2, L1.3
- net N$29: now also C4.1, U$1.1; no longer C3.1, L1.1
- net NEUTRAL: now also U$1.4; no longer L1.4
Other:
- moved on the sheet: C3, L1
