File: 1.4/emonVS.sch (EAGLE design)
At the start: 46 parts, among them J7 RJ45 Jack, J8 TERMINAL_BLOCK_2P, J9 TERMINAL_BLOCK_5P, M1 275VAC, M2 275VAC, M3 275VAC, T1 ZMPT101B, T2 ZMPT101B, T3 ZMPT101B

Commit message: improved thermal, swap around earth neutral, 0R link option
Parts:
- added R7: 0R, My-RLC:R_1206
Connections:
- removed net N$28: C4.2, J9-2.P$1, M1.1, M2.1, M3.1, U$1.3
- new net N$17: C4.2, J9-1.P$1, M1.1, M2.1, M3.1, U$1.3
- new net N$20: J9-2.P$1, R7.2
- net GND: now also R7.1; no longer J9-1.P$1
Changed lines of the file:
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@@
 <setting verticaltext="up"/>
 </settings>
-<grid distance="0.1" unitdist="inch" unit="inch" style="lines" multiple="1" display="no" altdistance="0.01" altunitdist="inch" altunit="inch"/>
+<grid distance="0.025" unitdist="inch" unit="inch" style="lines" multiple="1" display="no" altdistance="0.01" altunitdist="inch" altunit="inch"/>
 <layers>
 <layer number="1" name="Top" color="59" fill="1" visible="no" active="no"/>
@@
 <part name="SUPPLY7" library="My-Supply" library_urn="urn:adsk.eagle:library:35531236" deviceset="0V" device=""/>
 <part name="SUPPLY8" library="My-Supply" library_urn="urn:adsk.eagle:library:35531236" deviceset="5V" device=""/>
+<part name="R7" library="My-RLC" library_urn="urn:adsk.eagle:library:35509816" deviceset="R_" device="1206" package3d_urn="urn:adsk.eagle:package:35509967/1" value="0R">
+<attribute name="PN" value="ERJ-H3GJ103V"/>
+</part>
 </parts>
 <sheets>
@@
 <attribute name="VALUE" x="178.4096" y="119.38" size="1.27" layer="96" rot="MR0" align="center"/>
 </instance>
+<instance part="R7" gate="G$1" x="25.4" y="125.095" smashed="yes" rot="MR0">
+<attribute name="PN" x="25.4" y="125.095" size="1.778" layer="96" display="off"/>
+<attribute name="NAME" x="25.4" y="127.2286" size="1.27" layer="95" rot="MR0" align="center"/>
+<attribute name="VALUE" x="25.4" y="123.19" size="1.27" layer="96" rot="MR0" align="center"/>
+</instance>
 </instances>
 <busses>
@@
 <wire x1="18.415" y1="151.765" x2="21.59" y2="151.765" width="0.1524" layer="91" grouprefs="THREE-PHASE_AC_NETWORK_INTERFACE"/>
 <pinref part="J9" gate="-4" pin="P$1"/>
-</segment>
-</net>
-<net name="N$28" class="0">
-<segment>
-<wire x1="90.17" y1="125.095" x2="80.01" y2="125.095" width="0.1524" layer="91" grouprefs="THREE-PHASE_AC_NETWORK_INTERFACE"/>
-<pinref part="J9" gate="-2" pin="P$1"/>
-<pinref part="C4" gate="G$1" pin="2"/>
-<wire x1="80.01" y1="125.095" x2="66.04" y2="125.095" width="0.1524" layer="91" grouprefs="THREE-PHASE_AC_NETWORK_INTERFACE"/>
-<wire x1="66.04" y1="125.095" x2="53.34" y2="125.095" width="0.1524" layer="91" grouprefs="THREE-PHASE_AC_NETWORK_INTERFACE"/>
-<wire x1="53.34" y1="125.095" x2="40.64" y2="125.095" width="0.1524" layer="91" grouprefs="THREE-PHASE_AC_NETWORK_INTERFACE"/>
-<wire x1="40.64" y1="125.095" x2="18.415" y2="125.095" width="0.1524" layer="91" grouprefs="THREE-PHASE_AC_NETWORK_INTERFACE"/>
-<wire x1="80.01" y1="129.54" x2="80.01" y2="125.095" width="0.1524" layer="91" grouprefs="THREE-PHASE_AC_NETWORK_INTERFACE"/>
-<junction x="80.01" y="125.095" grouprefs="THREE-PHASE_AC_NETWORK_INTERFACE"/>
-<pinref part="U$1" gate="G$1" pin="3"/>
-<wire x1="93.345" y1="130.81" x2="90.17" y2="130.81" width="0.1524" layer="91" grouprefs="THREE-PHASE_AC_NETWORK_INTERFACE"/>
-<wire x1="90.17" y1="130.81" x2="90.17" y2="125.095" width="0.1524" layer="91" grouprefs="THREE-PHASE_AC_NETWORK_INTERFACE"/>
-<pinref part="M1" gate="G$1" pin="1"/>
-<wire x1="40.64" y1="127" x2="40.64" y2="125.095" width="0.1524" layer="91" grouprefs="THREE-PHASE_AC_NETWORK_INTERFACE"/>
-<junction x="40.64" y="125.095" grouprefs="THREE-PHASE_AC_NETWORK_INTERFACE"/>
-<pinref part="M2" gate="G$1" pin="1"/>
-<wire x1="53.34" y1="127.635" x2="53.34" y2="125.095" width="0.1524" layer="91" grouprefs="THREE-PHASE_AC_NETWORK_INTERFACE"/>
-<junction x="53.34" y="125.095" grouprefs="THREE-PHASE_AC_NETWORK_INTERFACE"/>
-<pinref part="M3" gate="G$1" pin="1"/>
-<wire x1="66.04" y1="127.635" x2="66.04" y2="125.095" width="0.1524" layer="91" grouprefs="THREE-PHASE_AC_NETWORK_INTERFACE"/>
-<junction x="66.04" y="125.095" grouprefs="THREE-PHASE_AC_NETWORK_INTERFACE"/>
 </segment>
 </net>
@@
 </segment>
 <segment>
-<wire x1="18.415" y1="114.935" x2="59.69" y2="114.935" width="0.1524" layer="91" grouprefs="THREE-PHASE_AC_NETWORK_INTERFACE"/>
 <label x="114.3" y="114.935" size="1.27" layer="95" xref="yes" grouprefs="THREE-PHASE_AC_NETWORK_INTERFACE"/>
-<pinref part="J9" gate="-1" pin="P$1"/>
 <pinref part="SUPPLY6" gate="G$1" pin="0V"/>
 <wire x1="59.69" y1="114.935" x2="114.3" y2="114.935" width="0.1524" layer="91" grouprefs="THREE-PHASE_AC_NETWORK_INTERFACE"/>
 <wire x1="59.69" y1="113.03" x2="59.69" y2="114.935" width="0.1524" layer="91" grouprefs="THREE-PHASE_AC_NETWORK_INTERFACE"/>
-<junction x="59.69" y="114.935" grouprefs="THREE-PHASE_AC_NETWORK_INTERFACE"/>
+<pinref part="R7" gate="G$1" pin="1"/>
+<wire x1="30.48" y1="125.095" x2="30.48" y2="116.84" width="0.1524" layer="91"/>
+<wire x1="30.48" y1="116.84" x2="59.69" y2="116.84" width="0.1524" layer="91"/>
+<wire x1="59.69" y1="116.84" x2="59.69" y2="114.935" width="0.1524" layer="91"/>
+<junction x="59.69" y="114.935"/>
 </segment>
 <segment>
@@
 </segment>
 </net>
+<net name="N$17" class="0">
+<segment>
+<pinref part="J9" gate="-1" pin="P$1"/>
+<wire x1="18.415" y1="114.935" x2="18.415" y2="114.3" width="0.1524" layer="91"/>
+<wire x1="18.415" y1="114.3" x2="40.64" y2="114.3" width="0.1524" layer="91"/>
+<wire x1="40.64" y1="114.3" x2="40.64" y2="125.095" width="0.1524" layer="91"/>
+<wire x1="90.17" y1="125.095" x2="80.01" y2="125.095" width="0.1524" layer="91" grouprefs="THREE-PHASE_AC_NETWORK_INTERFACE"/>
+<pinref part="C4" gate="G$1" pin="2"/>
+<wire x1="80.01" y1="125.095" x2="66.04" y2="125.095" width="0.1524" layer="91" grouprefs="THREE-PHASE_AC_NETWORK_INTERFACE"/>
+<wire x1="66.04" y1="125.095" x2="53.34" y2="125.095" width="0.1524" layer="91" grouprefs="THREE-PHASE_AC_NETWORK_INTERFACE"/>
+<wire x1="53.34" y1="125.095" x2="40.64" y2="125.095" width="0.1524" layer="91" grouprefs="THREE-PHASE_AC_NETWORK_INTERFACE"/>
+<wire x1="80.01" y1="129.54" x2="80.01" y2="125.095" width="0.1524" layer="91" grouprefs="THREE-PHASE_AC_NETWORK_INTERFACE"/>
+<junction x="80.01" y="125.095" grouprefs="THREE-PHASE_AC_NETWORK_INTERFACE"/>
+<pinref part="U$1" gate="G$1" pin="3"/>
+<wire x1="93.345" y1="130.81" x2="90.17" y2="130.81" width="0.1524" layer="91" grouprefs="THREE-PHASE_AC_NETWORK_INTERFACE"/>
+<wire x1="90.17" y1="130.81" x2="90.17" y2="125.095" width="0.1524" layer="91" grouprefs="THREE-PHASE_AC_NETWORK_INTERFACE"/>
+<pinref part="M1" gate="G$1" pin="1"/>
+<wire x1="40.64" y1="127" x2="40.64" y2="125.095" width="0.1524" layer="91" grouprefs="THREE-PHASE_AC_NETWORK_INTERFACE"/>
+<pinref part="M2" gate="G$1" pin="1"/>
+<wire x1="53.34" y1="127.635" x2="53.34" y2="125.095" width="0.1524" layer="91" grouprefs="THREE-PHASE_AC_NETWORK_INTERFACE"/>
+<junction x="53.34" y="125.095" grouprefs="THREE-PHASE_AC_NETWORK_INTERFACE"/>
+<pinref part="M3" gate="G$1" pin="1"/>
+<wire x1="66.04" y1="127.635" x2="66.04" y2="125.095" width="0.1524" layer="91" grouprefs="THREE-PHASE_AC_NETWORK_INTERFACE"/>
+<junction x="66.04" y="125.095" grouprefs="THREE-PHASE_AC_NETWORK_INTERFACE"/>
+<junction x="40.64" y="125.095"/>
+</segment>
+</net>
+<net name="N$20" class="0">
+<segment>
+<pinref part="J9" gate="-2" pin="P$1"/>
+<pinref part="R7" gate="G$1" pin="2"/>
+<wire x1="18.415" y1="125.095" x2="20.32" y2="125.095" width="0.1524" layer="91"/>
+</segment>
+</net>
